Commit message: spin up realsense camera in sim

File: urdf/_d435.gazebo.xacro (robot description, xacro)
@@ -23,10 +23,22 @@
       <!--<max_vel>0.01</max_vel>
       <min_depth>0</min_depth>-->
-      <sensor name="${camera_name}color" type="camera">
-        <camera name="${camera_name}">
+      <sensor name="custom_camera_rgbd" type="rgbd_camera">
+        <always_on>1</always_on>
+        <update_rate>30</update_rate>
+        <visualize>1</visualize>
+        <topic>custom_topic/color</topic>
+        <enable_metrics>1</enable_metrics>
+        <plugin filename="libignition-gazebo-sensors-system.so"
+        name="ignition::gazebo::systems::Sensors"/>
+        <camera name="$custom_camera/color">
+          <triggered>0</triggered>
+          <camera_info_topic>custom_camera/camera_info</camera_info_topic>
           <horizontal_fov>${69.4*deg_to_rad}</horizontal_fov>
+          <save enabled="true">
+            <path>/ros2_ws/src</path>
+          </save>
           <image>
-            <width>640</width>
-            <height>480</height>
+            <width>320</width>
+            <height>240</height>
             <format>RGB_INT8</format>
           </image>
@@ -40,59 +52,13 @@
             <stddev>0.007</stddev>
           </noise>
+          <depth_camera>
+            <output>custom_depths</output>
+          </depth_camera>
         </camera>
-        <always_on>1</always_on>
-        <update_rate>30</update_rate>
-        <visualize>1</visualize>
-      </sensor>
-      <sensor name="${camera_name}ired1" type="camera">
-        <camera name="${camera_name}">
+        <camera name="${camera_name}depth">
           <horizontal_fov>${85.2*deg_to_rad}</horizontal_fov>
           <image>
-            <width>1280</width>
-            <height>720</height>
-            <format>L_INT8</format>
-          </image>
-          <clip>
-            <near>0.1</near>
-            <far>100</far>
-          </clip>
-          <noise>
-            <type>gaussian</type>
-            <mean>0.0</mean>
-            <stddev>0.05</stddev>
-          </noise>
-        </camera>
-        <always_on>1</always_on>
-        <update_rate>90</update_rate>
-        <visualize>0</visualize>
-      </sensor>
-      <sensor name="${camera_name}ired2" type="camera">
-        <camera name="${camera_name}">
-          <horizontal_fov>${85.2*deg_to_rad}</horizontal_fov>
-          <image>
-            <width>1280</width>
-            <height>720</height>
-            <format>L_INT8</format>
-          </image>
-          <clip>
-            <near>0.1</near>
-            <far>100</far>
-          </clip>
-          <noise>
-            <type>gaussian</type>
-            <mean>0.0</mean>
-            <stddev>0.05</stddev>
-          </noise>
-        </camera>
-        <always_on>1</always_on>
-        <update_rate>90</update_rate>
-        <visualize>0</visualize>
-      </sensor>
-      <sensor name="${camera_name}depth" type="depth">
-        <camera name="${camera_name}">
-          <horizontal_fov>${85.2*deg_to_rad}</horizontal_fov>
-          <image>
-            <width>1280</width>
-            <height>720</height>
+            <width>320</width>
+            <height>240</height>
           </image>
           <clip>
@@ -106,34 +72,15 @@
           </noise>
         </camera>
-        <always_on>1</always_on>
-        <update_rate>90</update_rate>
-        <visualize>0</visualize>
+        <point_cloud>
+          <topic>custom_name/points</topic>
+          <sample_rate>2</sample_rate>
+        </point_cloud>
       </sensor>
-    </gazebo>
-    <gazebo>
-      <plugin name="${topics_ns}" filename="librealsense_gazebo_plugin.so">
-        <prefix>${camera_name}</prefix>
-        <depthUpdateRate>30.0</depthUpdateRate>
-        <colorUpdateRate>30.0</colorUpdateRate>
-        <infraredUpdateRate>30.0</infraredUpdateRate>
-        <depthTopicName>depth/image_raw</depthTopicName>
-        <depthCameraInfoTopicName>depth/camera_info</depthCameraInfoTopicName>
-        <colorTopicName>color/image_raw</colorTopicName>
-        <colorCameraInfoTopicName>color/camera_info</colorCameraInfoTopicName>
-        <infrared1TopicName>infra1/image_raw</infrared1TopicName>
-        <infrared1CameraInfoTopicName>infra1/camera_info</infrared1CameraInfoTopicName>
-        <infrared2TopicName>infra2/image_raw</infrared2TopicName>
-        <infrared2CameraInfoTopicName>infra2/camera_info</infrared2CameraInfoTopicName>
-        <colorOpticalframeName>${color_optical_frame}</colorOpticalframeName>
-        <depthOpticalframeName>${depth_optical_frame}</depthOpticalframeName>
-        <infrared1OpticalframeName>${infrared1_optical_frame}</infrared1OpticalframeName>
-        <infrared2OpticalframeName>${infrared2_optical_frame}</infrared2OpticalframeName>
-        <rangeMinDepth>0.2</rangeMinDepth>
-        <rangeMaxDepth>10.0</rangeMaxDepth>
-        <pointCloud>${publish_pointcloud}</pointCloud>
-        <pointCloudTopicName>depth/color/points</pointCloudTopicName>
-        <pointCloudCutoff>0.25</pointCloudCutoff>
-        <pointCloudCutoffMax>9.0</pointCloudCutoffMax>
-      </plugin>
+              <point_cloud>
+          <topic>custom_name/points</topic>
+          <sample_rate>2</sample_rate>
+        </point_cloud>
+        <plugin filename="libignition-gazebo-sensors-system.so"
+        name="ignition::gazebo::systems::Sensors"/>
     </gazebo>
   </xacro:macro>

File: urdf/_d435.urdf.xacro (robot description, xacro)
@@ -47,6 +47,6 @@
       <origin xyz="${d435_cam_mount_from_center_offset} ${-d435_cam_depth_py} 0" rpy="${M_PI/2} 0 ${M_PI/2}"/>
         <geometry>
-          <!-- <box size="${d435_cam_width} ${d435_cam_height} ${d435_cam_depth}"/> -->
-          <mesh filename="package://realsense2_description/meshes/d435.dae" />
+          <box size="${d435_cam_width} ${d435_cam_height} ${d435_cam_depth}"/>
+          <!-- <mesh filename="$(find realsense2_description)/meshes/d435.dae" /> -->
           <!--<mesh filename="package://realsense2_description/meshes/d435/d435.dae" />-->
         </geometry>

Commit message: linked pointcloud sim to octomap

File: urdf/_d435.gazebo.xacro (robot description, xacro)
@@ -45,5 +45,5 @@
           <clip>
             <near>0.1</near>
-            <far>100</far>
+            <far>5</far>
           </clip>
           <noise>

File: urdf/_d435.urdf.xacro (robot description, xacro)
@@ -47,7 +47,7 @@
       <origin xyz="${d435_cam_mount_from_center_offset} ${-d435_cam_depth_py} 0" rpy="${M_PI/2} 0 ${M_PI/2}"/>
         <geometry>
-          <box size="${d435_cam_width} ${d435_cam_height} ${d435_cam_depth}"/>
-          <!-- <mesh filename="$(find realsense2_description)/meshes/d435.dae" /> -->
-          <!--<mesh filename="package://realsense2_description/meshes/d435/d435.dae" />-->
+          <!-- <box size="${d435_cam_width} ${d435_cam_height} ${d435_cam_depth}"/> -->
+          <mesh filename="file:$(find realsense2_description)/meshes/d435.dae" />
+          <!-- <mesh filename="model://realsense2_description/meshes/d435/d435.dae" /> -->
         </geometry>
         <material name="${name}_aluminum"/>
